File: PCB/PCB_kicad/PCB_kicad.kicad_sch (KiCad schematic)
At the start: 21 parts, among them J1 Conn_01x15_Socket, J10 Conn_01x02_Socket, J11 Conn_01x04_Socket, J2 Conn_01x15_Socket, J3 Barrel_Jack_Switch_Pin3Ring, J4 Conn_01x08_Socket, J5 Conn_01x04_Socket, J6 Conn_01x04_Socket, J7 Conn_01x04_Socket, J8 Conn_01x04_Socket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

Commit message: Improved stability
Added some minor tweaks to improve the stability of the desing
Parts:
- J1, J2: footprint Connector_PinHeader_2.00mm:PinHeader_1x15_P2.00mm_Vertical -> Connector_PinHeader_2.54mm:PinHeader_1x15_P2.54mm_Vertical
Changed lines of the file:
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@@
 			)
 		)
-		(property "Footprint" "Connector_PinHeader_2.00mm:PinHeader_1x15_P2.00mm_Vertical"
+		(property "Footprint" "Connector_PinHeader_2.54mm:PinHeader_1x15_P2.54mm_Vertical"
 			(at 59.69 41.91 0)
 			(effects
@@
 			)
 		)
-		(property "Footprint" "Connector_PinHeader_2.00mm:PinHeader_1x15_P2.00mm_Vertical"
+		(property "Footprint" "Connector_PinHeader_2.54mm:PinHeader_1x15_P2.54mm_Vertical"
 			(at 36.83 41.91 0)
 			(effects
